Commit message: Feature: Use "$(find)" to get meshes to fix mesh loading issue

File: lbr_description/urdf/iiwa7/iiwa7_description.xacro (robot description, xacro)
@@ -31,5 +31,5 @@
                 <origin rpy="0 0 0" xyz="0 0 0" />
                 <geometry>
-                    <mesh filename="package://lbr_description/meshes/iiwa7/visual/link_0.dae" />
+                    <mesh filename="file://$(find lbr_description)/meshes/iiwa7/visual/link_0.dae" />
                 </geometry>
             </visual>
@@ -37,5 +37,5 @@
                 <origin rpy="0 0 0" xyz="0 0 0" />
                 <geometry>
-                    <mesh filename="package://lbr_description/meshes/iiwa7/collision/link_0.stl" />
+                    <mesh filename="file://$(find lbr_description)/meshes/iiwa7/collision/link_0.stl" />
                 </geometry>
             </collision>
@@ -63,5 +63,5 @@
                 <origin rpy="0 0 0" xyz="0.0 0.0 -0.1475" />
                 <geometry>
-                    <mesh filename="package://lbr_description/meshes/iiwa7/visual/link_1.dae" />
+                    <mesh filename="file://$(find lbr_description)/meshes/iiwa7/visual/link_1.dae" />
                 </geometry>
             </visual>
@@ -69,5 +69,5 @@
                 <origin rpy="0 0 0" xyz="0.0 0.0 -0.1475" />
                 <geometry>
-                    <mesh filename="package://lbr_description/meshes/iiwa7/collision/link_1.stl" />
+                    <mesh filename="file://$(find lbr_description)/meshes/iiwa7/collision/link_1.stl" />
                 </geometry>
             </collision>
@@ -95,5 +95,5 @@
                 <origin rpy="0 0 0" xyz="0.0 0.0105 -0.34" />
                 <geometry>
-                    <mesh filename="package://lbr_description/meshes/iiwa7/visual/link_2.dae" />
+                    <mesh filename="file://$(find lbr_description)/meshes/iiwa7/visual/link_2.dae" />
                 </geometry>
             </visual>
@@ -101,5 +101,5 @@
                 <origin rpy="0 0 0" xyz="0.0 0.0105 -0.34" />
                 <geometry>
-                    <mesh filename="package://lbr_description/meshes/iiwa7/collision/link_2.stl" />
+                    <mesh filename="file://$(find lbr_description)/meshes/iiwa7/collision/link_2.stl" />
                 </geometry>
             </collision>
@@ -127,5 +127,5 @@
                 <origin rpy="0 0 0" xyz="0.0 0.0 -0.5475" />
                 <geometry>
-                    <mesh filename="package://lbr_description/meshes/iiwa7/visual/link_3.dae" />
+                    <mesh filename="file://$(find lbr_description)/meshes/iiwa7/visual/link_3.dae" />
                 </geometry>
             </visual>
@@ -133,5 +133,5 @@
                 <origin rpy="0 0 0" xyz="0.0 0.0 -0.5475" />
                 <geometry>
-                    <mesh filename="package://lbr_description/meshes/iiwa7/collision/link_3.stl" />
+                    <mesh filename="file://$(find lbr_description)/meshes/iiwa7/collision/link_3.stl" />
                 </geometry>
             </collision>
@@ -159,5 +159,5 @@
                 <origin rpy="0 0 0" xyz="0.0 -0.0105 -0.74" />
                 <geometry>
-                    <mesh filename="package://lbr_description/meshes/iiwa7/visual/link_4.dae" />
+                    <mesh filename="file://$(find lbr_description)/meshes/iiwa7/visual/link_4.dae" />
                 </geometry>
             </visual>
@@ -165,5 +165,5 @@
                 <origin rpy="0 0 0" xyz="0.0 -0.0105 -0.74" />
                 <geometry>
-                    <mesh filename="package://lbr_description/meshes/iiwa7/collision/link_4.stl" />
+                    <mesh filename="file://$(find lbr_description)/meshes/iiwa7/collision/link_4.stl" />
                 </geometry>
             </collision>
@@ -191,5 +191,5 @@
                 <origin rpy="0 0 0" xyz="0.0 0.0 -0.9475" />
                 <geometry>
-                    <mesh filename="package://lbr_description/meshes/iiwa7/visual/link_5.dae" />
+                    <mesh filename="file://$(find lbr_description)/meshes/iiwa7/visual/link_5.dae" />
                 </geometry>
             </visual>
@@ -197,5 +197,5 @@
                 <origin rpy="0 0 0" xyz="0.0 0.0 -0.9475" />
                 <geometry>
-                    <mesh filename="package://lbr_description/meshes/iiwa7/collision/link_5.stl" />
+                    <mesh filename="file://$(find lbr_description)/meshes/iiwa7/collision/link_5.stl" />
                 </geometry>
             </collision>
@@ -223,5 +223,5 @@
                 <origin rpy="0 0 0" xyz="0.0 0.0707 -1.14" />
                 <geometry>
-                    <mesh filename="package://lbr_description/meshes/iiwa7/visual/link_6.dae" />
+                    <mesh filename="file://$(find lbr_description)/meshes/iiwa7/visual/link_6.dae" />
                 </geometry>
             </visual>
@@ -229,5 +229,5 @@
                 <origin rpy="0 0 0" xyz="0.0 0.0707 -1.14" />
                 <geometry>
-                    <mesh filename="package://lbr_description/meshes/iiwa7/collision/link_6.stl" />
+                    <mesh filename="file://$(find lbr_description)/meshes/iiwa7/collision/link_6.stl" />
                 </geometry>
             </collision>
@@ -254,5 +254,5 @@
                 <origin rpy="0 0 0" xyz="0.0 0.0 -1.231" />
                 <geometry>
-                    <mesh filename="package://lbr_description/meshes/iiwa7/visual/link_7.dae" />
+                    <mesh filename="file://$(find lbr_description)/meshes/iiwa7/visual/link_7.dae" />
                 </geometry>
             </visual>
@@ -260,5 +260,5 @@
                 <origin rpy="0 0 0" xyz="0.0 0.0 -1.231" />
                 <geometry>
-                    <mesh filename="package://lbr_description/meshes/iiwa7/collision/link_7.stl" />
+                    <mesh filename="file://$(find lbr_description)/meshes/iiwa7/collision/link_7.stl" />
                 </geometry>
             </collision>
