Commit message: Add conditional handling for urdf xacro

File: lbr_description/urdf/iiwa7_gripper/iiwa7_gripper.xacro (robot description, xacro)
@@ -18,4 +18,11 @@
         <child link="link_0" />
     </joint>
+    <xacro:property name="use_sim" value="$(arg mode)" />
+    <xacro:if value="${use_sim == 'gazebo'}">
+        <xacro:property name="sim" value="true" />
+    </xacro:if>
+    <xacro:unless value="${use_sim == 'gazebo'}">
+        <xacro:property name="sim" value="false" />
+    </xacro:unless>
     <!-- iiwa -->
     <xacro:iiwa7
@@ -23,5 +30,5 @@
         mode="$(arg mode)"
         system_parameters_path="$(arg system_parameters_path)" />
-        <xacro:robotiq_gripper name="RobotiqGripperHardwareInterface" prefix="" parent="link_ee" use_fake_hardware="true">
+        <xacro:robotiq_gripper name="RobotiqGripperHardwareInterface" prefix="" parent="link_ee" use_fake_hardware="true" sim_ignition="${sim}">
         <origin xyz="0 0 0" rpy="0 0 0" />
         </xacro:robotiq_gripper>

Commit message: Refactor: Keep sane names for gripper parameters

File: lbr_description/urdf/iiwa7_gripper/iiwa7_gripper.xacro (robot description, xacro)
@@ -18,10 +18,16 @@
         <child link="link_0" />
     </joint>
-    <xacro:property name="use_sim" value="$(arg mode)" />
-    <xacro:if value="${use_sim == 'gazebo'}">
-        <xacro:property name="sim" value="true" />
+    <xacro:property name="operation_mode" value="$(arg mode)" />
+    <xacro:if value="${operation_mode == 'gazebo'}">
+        <xacro:property name="use_sim" value="true" />
     </xacro:if>
-    <xacro:unless value="${use_sim == 'gazebo'}">
-        <xacro:property name="sim" value="false" />
+    <xacro:unless value="${operation_mode == 'gazebo'}">
+        <xacro:property name="use_sim" value="false" />
+    </xacro:unless>
+    <xacro:if value="${operation_mode == 'mock'}">
+        <xacro:property name="fake_hardware" value="true" />
+    </xacro:if>
+    <xacro:unless value="${operation_mode == 'mock'}">
+        <xacro:property name="fake_hardware" value="false" />
     </xacro:unless>
     <!-- iiwa -->
@@ -30,5 +36,5 @@
         mode="$(arg mode)"
         system_parameters_path="$(arg system_parameters_path)" />
-        <xacro:robotiq_gripper name="RobotiqGripperHardwareInterface" prefix="" parent="link_ee" use_fake_hardware="true" sim_ignition="true">
+        <xacro:robotiq_gripper name="RobotiqGripperHardwareInterface" prefix="" parent="link_ee" use_fake_hardware="${fake_hardware}" sim_ignition="${use_sim}">
         <origin xyz="0 0 0" rpy="0 0 0" />
         </xacro:robotiq_gripper>

Commit message: Feature: Add realsense d415 to gripper (no mounting bracket though :( )

File: lbr_description/urdf/iiwa7_gripper/iiwa7_gripper.xacro (robot description, xacro)
@@ -5,4 +5,5 @@
     <xacro:include filename="$(find lbr_description)/urdf/iiwa7/iiwa7_description.xacro" />
     <xacro:include filename="$(find robotiq_description)/urdf/robotiq_2f_85_macro.urdf.xacro"/>
+    <xacro:include filename="$(find gazebo_sensor_collection)/urdf/cameras/rgbd/realsense_d415.urdf.xacro" />
     <xacro:arg name="robot_name" default="lbr" />
     <xacro:arg name="mode" default="mock" />
@@ -36,6 +37,9 @@
         mode="$(arg mode)"
         system_parameters_path="$(arg system_parameters_path)" />
-        <xacro:robotiq_gripper name="RobotiqGripperHardwareInterface" prefix="" parent="link_ee" use_fake_hardware="${fake_hardware}" sim_ignition="${use_sim}">
+    <xacro:robotiq_gripper name="RobotiqGripperHardwareInterface" prefix="" parent="link_ee" use_fake_hardware="${fake_hardware}" sim_ignition="${use_sim}">
         <origin xyz="0 0 0" rpy="0 0 0" />
-        </xacro:robotiq_gripper>
+    </xacro:robotiq_gripper>
+    <xacro:sensor_realsense_d415 name="real_sense" parent="link_ee">
+        <origin xyz="0 0.05 0.03 " rpy="0 -1.57079 -1.57079" />
+    </xacro:sensor_realsense_d415>
 </robot>
